Commit message: ros2_control

File: install/vox/share/vox/description/colors.xacro (robot description, xacro)
@@ -1 +1 @@
-/home/vox/Desktop/vox/src/description/colors.xacro
+/home/claw/Desktop/Vox/src/description/colors.xacro

File: install/vox/share/vox/description/robot.urdf.xacro (robot description, xacro)
@@ -1 +1 @@
-/home/vox/Desktop/vox/src/description/robot.urdf.xacro
+/home/claw/Desktop/Vox/src/description/robot.urdf.xacro

File: install/vox/share/vox/description/robot_core.xacro (robot description, xacro)
@@ -1 +1 @@
-/home/vox/Desktop/vox/src/description/robot_core.xacro
+/home/claw/Desktop/Vox/src/description/robot_core.xacro

File: src/description/robot.urdf.xacro (robot description, xacro)
@@ -2,3 +2,7 @@
 <robot xmlns:xacro="http://www.ros.org/wiki/xacro" name="vox">
 	<xacro:include filename="robot_core.xacro"/>
+	<!-- <xacro:include filename="gazebo_controls.xacro"/> -->
+	<xacro:include filename="ros2_control.xacro"/>
+	<xacro:include filename="laser.xacro"/>
+	<xacro:include filename="camera.xacro"/>
 </robot>

File: src/description/robot_core.xacro (robot description, xacro)
@@ -32,4 +32,7 @@
         </inertial>
     </link>
+    <gazebo reference="chassis">
+        <material>Gazebo/White</material>
+    </gazebo>
     <joint name="front_left_wheel_joint" type="continuous">
         <parent link="chassis"/>
@@ -38,5 +41,4 @@
         <axis xyz="0 0 1"/>
     </joint>
-0
     <link name="front_left_wheel">
         <visual>
@@ -61,4 +63,7 @@
         </inertial>
     </link>
+    <gazebo reference="front_left_wheel">
+        <material>Gazebo/Blue</material>
+    </gazebo>
     <joint name="front_right_wheel_joint" type="continuous">
         <parent link="chassis"/>
@@ -89,4 +94,7 @@
         </inertial>
     </link>
+    <gazebo reference="front_right_wheel">
+        <material>Gazebo/Blue</material>
+    </gazebo>
     <joint name="back_left_wheel_joint" type="continuous">
         <parent link="chassis"/>
@@ -95,5 +103,4 @@
         <axis xyz="0 0 1"/>
     </joint>
-0
     <link name="back_left_wheel">
         <visual>
@@ -118,4 +125,7 @@
         </inertial>
     </link>
+    <gazebo reference="back_left_wheel">
+        <material>Gazebo/Blue</material>
+    </gazebo>
     <joint name="back_right_wheel_joint" type="continuous">
         <parent link="chassis"/>
@@ -146,3 +156,6 @@
         </inertial>
     </link>
+    <gazebo reference="back_right_wheel">
+        <material>Gazebo/Blue</material>
+    </gazebo>
 </robot>
