Commit message: adding all 4 wheel drive + some docs used in some tries to fix the rviz gezebo desync

File: install/vox/share/vox/description/camera.xacro (robot description, xacro)
@@ -1 +1 @@
-/home/claw/Desktop/Vox/src/description/camera.xacro
+/home/vox/Desktop/Vox/src/description/camera.xacro

File: install/vox/share/vox/description/colors.xacro (robot description, xacro)
@@ -1 +1 @@
-/home/claw/Desktop/Vox/src/description/colors.xacro
+/home/vox/Desktop/Vox/src/description/colors.xacro

File: install/vox/share/vox/description/gazebo_controls.xacro (robot description, xacro)
@@ -1 +1 @@
-/home/claw/Desktop/Vox/src/description/gazebo_controls.xacro
+/home/vox/Desktop/Vox/src/description/gazebo_controls.xacro

File: install/vox/share/vox/description/laser.xacro (robot description, xacro)
@@ -1 +1 @@
-/home/claw/Desktop/Vox/src/description/laser.xacro
+/home/vox/Desktop/Vox/src/description/laser.xacro

File: install/vox/share/vox/description/robot.urdf.xacro (robot description, xacro)
@@ -1 +1 @@
-/home/claw/Desktop/Vox/src/description/robot.urdf.xacro
+/home/vox/Desktop/Vox/src/description/robot.urdf.xacro

File: install/vox/share/vox/description/robot_core.xacro (robot description, xacro)
@@ -1 +1 @@
-/home/claw/Desktop/Vox/src/description/robot_core.xacro
+/home/vox/Desktop/Vox/src/description/robot_core.xacro

File: install/vox/share/vox/description/ros2_control.xacro (robot description, xacro)
@@ -1 +1 @@
-/home/claw/Desktop/Vox/src/description/ros2_control.xacro
+/home/vox/Desktop/Vox/src/description/ros2_control.xacro

File: src/description/gazebo_controls.xacro (robot description, xacro)
@@ -4,7 +4,7 @@
 		<plugin name="diff_drive" filename="libgazebo_ros_diff_drive.so">
 			<left_joint>front_left_wheel_joint</left_joint>
-			<left_joint>back_left_wheel_joint</left_joint>
+			<!-- <left_joint>back_left_wheel_joint</left_joint> -->
 			<right_joint>front_right_wheel_joint</right_joint>
-			<right_joint>back_right_wheel_joint</right_joint>
+			<!-- <right_joint>back_right_wheel_joint</right_joint> -->
 			<wheel_separation>0.229</wheel_separation>
 			<wheel_diameter>0.12</wheel_diameter>

File: src/description/ros2_control.xacro (robot description, xacro)
@@ -6,4 +6,12 @@
 		</hardware>
 		<joint name="front_left_wheel_joint">
+			<command_interface name="velocity">
+				<param name="min">-10</param>
+				<param name="max">10</param>
+			</command_interface>
+			<state_interface name="velocity"></state_interface>
+			<state_interface name="position"></state_interface>
+		</joint>
+		<joint name="back_left_wheel_joint">
 			<command_interface name="velocity">
 				<param name="min">-10</param>
@@ -21,5 +29,13 @@
 			<state_interface name="position"></state_interface>
 		</joint>
-		</ros2_control>
+		<joint name="back_right_wheel_joint">
+			<command_interface name="velocity">
+				<param name="min">-10</param>
+				<param name="max">10</param>
+			</command_interface>
+			<state_interface name="velocity"></state_interface>
+			<state_interface name="position"></state_interface>
+		</joint>
+	</ros2_control>
 	<gazebo>
 		<plugin name="gazebo_ros2_control" filename="libgazebo_ros2_control.so">
