Commit message: tweaks to the simulations

File: src/description/robot.urdf.xacro (robot description, xacro)
@@ -1,7 +1,12 @@
 <?xml version="1.0"?>
 <robot xmlns:xacro="http://www.ros.org/wiki/xacro" name="vox">
+	<xacro:arg name="use_ros2_control" default="true"/>
 	<xacro:include filename="robot_core.xacro"/>
-	<!-- <xacro:include filename="gazebo_controls.xacro"/> -->
-	<xacro:include filename="ros2_control.xacro"/>
+	<xacro:if value="$(arg use_ros2_control)">
+		<xacro:include filename="ros2_control.xacro"/>
+	</xacro:if>
+	<xacro:unless value="$(arg use_ros2_control)">
+		<xacro:include filename="gazebo_controls.xacro"/>
+	</xacro:unless>
 	<xacro:include filename="laser.xacro"/>
 	<xacro:include filename="camera.xacro"/>

File: src/description/robot_core.xacro (robot description, xacro)
@@ -50,5 +50,6 @@
         <collision>
             <geometry>
-                <cylinder radius="0.06" length="0.06"/>
+                <!-- <cylinder radius="0.06" length="0.06"/> -->
+                <sphere radius="0.06"/>
             </geometry>
         </collision>
@@ -81,5 +82,6 @@
         <collision>
             <geometry>
-                <cylinder radius="0.06" length="0.06"/>
+                <!-- <cylinder radius="0.06" length="0.06"/> -->
+                <sphere radius="0.06"/>
             </geometry>
         </collision>
@@ -112,5 +114,6 @@
         <collision>
             <geometry>
-                <cylinder radius="0.06" length="0.06"/>
+                <!-- <cylinder radius="0.06" length="0.06"/> -->
+                <sphere radius="0.06"/>
             </geometry>
         </collision>
@@ -143,5 +146,6 @@
         <collision>
             <geometry>
-                <cylinder radius="0.06" length="0.06"/>
+                <!-- <cylinder radius="0.06" length="0.06"/> -->
+                <sphere radius="0.06"/>
             </geometry>
         </collision>
