Commit message: added parameters for slam + CHECK COMMANDS.TXT for info + MAKE SURE TO BUILD IT WHEN YOU FIRST RUN IT

File: src/description/robot_core.xacro (robot description, xacro)
@@ -2,6 +2,14 @@
 <robot xmlns:xacro="http://www.ros.org/wiki/xacro">
     <xacro:include filename="colors.xacro"/>
-    <link name="base_link">
-    </link>
+    <!-- BASE LINK -->
+    <link name="base_link"></link>
+    <!-- BASE FOOTPRINT LINK -->
+    <joint name="base_footprint_joint" type="fixed">
+        <parent link="base_link"/>
+        <child link="base_footprint"/>
+        <origin xyz="0 0 0" rpy="0 0 0"/>
+    </joint>
+    <link name="base_footprint"></link>
+    <!-- CHASSIS LINK -->
     <joint name="chassis_joint" type="fixed">
         <parent link="base_link"/>
