Commit message: partially fixing drift between Gazebo and RViz

File: src/description/gazebo_controls.xacro (robot description, xacro)
@@ -2,18 +2,20 @@
 <robot xmlns:xacro="http://www.ros.org/wiki/xacro">
 	<gazebo>
-		<plugin name="diff_drive" filename="libgazebo_ros_diff_drive.so">
-			<left_joint>front_left_wheel_joint</left_joint>
-			<!-- <left_joint>back_left_wheel_joint</left_joint> -->
-			<right_joint>front_right_wheel_joint</right_joint>
-			<!-- <right_joint>back_right_wheel_joint</right_joint> -->
-			<wheel_separation>0.229</wheel_separation>
-			<wheel_diameter>0.12</wheel_diameter>
-			<max_wheel_torque>200</max_wheel_torque>
-			<max_wheel_acceleration>10.0</max_wheel_acceleration>
-			<odometry_frame>odom</odometry_frame>
-			<robot_base_frame>base_link</robot_base_frame>
-			<publish_odom>true</publish_odom>
-			<publish_odom_tf>true</publish_odom_tf>
-			<publish_wheel_tf>true</publish_wheel_tf>
+		<plugin name="skid_steer_drive_controller" filename="libgazebo_ros_skid_steer_drive.so">
+			<dds_domain_id>42</dds_domain_id>
+		    <topic_name_twist>cmd_vel</topic_name_twist>
+		    <topic_name_odometry>odom</topic_name_odometry>
+		    <topic_name_joint>joint</topic_name_joint>
+		    <right_front_joint>front_right_wheel_joint</right_front_joint>
+		    <right_rear_joint>back_right_wheel_joint</right_rear_joint>
+		    <left_front_joint>front_left_wheel_joint</left_front_joint>
+		    <left_rear_joint>back_left_wheel_joint</left_rear_joint>
+		    <wheel_separation>0.229</wheel_separation>
+		    <wheel_diameter>0.06</wheel_diameter>
+		    <wheel_torque>10</wheel_torque>
+		    <update_rate>2</update_rate>
+		    <covariance_x>0.0001</covariance_x>
+		    <covariance_y>0.0001</covariance_y>
+		    <covariance_yaw>0.01</covariance_yaw>
 		</plugin>
 	</gazebo>

File: src/description/laser.xacro (robot description, xacro)
@@ -9,5 +9,5 @@
 		<visual>
             <geometry>
-                <cylinder radius="0.06" length="0.06"/>
+                <cylinder radius="0.03" length="0.05"/>
             </geometry>
             <material name="blue"/>
@@ -22,7 +22,7 @@
             <mass value="0.17"/>
             <inertia
-                ixx="${(1/12) * 0.17 * (3*0.06*0.06 + 0.06*0.06)}" ixy="0.0" ixz="0.0"
-                iyy="${(1/12) * 0.17 * (3*0.06*0.06 + 0.06*0.06)}" iyz="0.0"
-                izz="${(1/12) * 0.17 * (0.06*0.06)}"
+                ixx="${0.17*(3*0.03*0.03+0.05*0.05)/12}" ixy="0.0" ixz="0.0"
+                iyy="${0.17*(3*0.03*0.03+0.05*0.05)/12}" iyz="0.0"
+                izz="${0.17*0.03*0.03/2}"
             />
         </inertial>

File: src/description/robot.urdf.xacro (robot description, xacro)
@@ -1,5 +1,5 @@
 <?xml version="1.0"?>
 <robot xmlns:xacro="http://www.ros.org/wiki/xacro" name="vox">
-	<xacro:arg name="use_ros2_control" default="true"/>
+	<xacro:arg name="use_ros2_control" default="false"/>
 	<xacro:include filename="robot_core.xacro"/>
 	<xacro:if value="$(arg use_ros2_control)">

File: src/description/robot_core.xacro (robot description, xacro)
@@ -34,7 +34,7 @@
             <mass value="0.67"/>
             <inertia
-                ixx="${(1/12) * 0.67 * (0.135*0.135+0.0475*0.0475)}" ixy="0.0" ixz="0.0"
-                iyy="${(1/12) * 0.67 * (0.21*0.21+0.0475*0.0475)}" iyz="0.0"
-                izz="${(1/12) * 0.67 * (0.21*0.21+0.135*0.135)}"
+                ixx="${0.67*(0.135*0.135+0.0475*0.0475)/12}" ixy="0.0" ixz="0.0"
+                iyy="${0.67*(0.21*0.21+0.0475*0.0475)/12}" iyz="0.0"
+                izz="${0.67*(0.21*0.21+0.135*0.135)/12}"
             />
         </inertial>
@@ -46,5 +46,5 @@
         <parent link="chassis"/>
         <child link="front_left_wheel"/>
-        <origin xyz="-0.08 0.1145 0" rpy="-${pi/2} 0 0"/>
+        <origin xyz="0.08 0.1145 0" rpy="-${pi/2} 0 0"/>
         <axis xyz="0 0 1"/>
     </joint>
@@ -66,7 +66,7 @@
             <mass value="0.17"/>
             <inertia
-                ixx="${(1/12) * 0.17 * (3*0.06*0.06 + 0.06*0.06)}" ixy="0.0" ixz="0.0"
-                iyy="${(1/12) * 0.17 * (3*0.06*0.06 + 0.06*0.06)}" iyz="0.0"
-                izz="${(1/12) * 0.17 * (0.06*0.06)}"
+                ixx="${0.17*(3*0.06*0.06+0.06*0.06)/12}" ixy="0.0" ixz="0.0"
+                iyy="${0.17*(3*0.06*0.06+0.06*0.06)/12}" iyz="0.0"
+                izz="${0.17*(0.06*0.06)/2}"
             />
         </inertial>
@@ -78,5 +78,5 @@
         <parent link="chassis"/>
         <child link="front_right_wheel"/>
-        <origin xyz="-0.08 -0.1145 0" rpy="${pi/2} 0 0"/>
+        <origin xyz="0.08 -0.1145 0" rpy="${pi/2} 0 0"/>
         <axis xyz="0 0 -1"/>
     </joint>
@@ -98,7 +98,7 @@
             <mass value="0.17"/>
             <inertia
-                ixx="${(1/12) * 0.17 * (3*0.06*0.06 + 0.06*0.06)}" ixy="0.0" ixz="0.0"
-                iyy="${(1/12) * 0.17 * (3*0.06*0.06 + 0.06*0.06)}" iyz="0.0"
-                izz="${(1/12) * 0.17 * (0.06*0.06)}"
+                ixx="${0.17*(3*0.06*0.06+0.06*0.06)/12}" ixy="0.0" ixz="0.0"
+                iyy="${0.17*(3*0.06*0.06+0.06*0.06)/12}" iyz="0.0"
+                izz="${0.17*(0.06*0.06)/2}"
             />
         </inertial>
@@ -110,5 +110,5 @@
         <parent link="chassis"/>
         <child link="back_left_wheel"/>
-        <origin xyz="0.08 0.1145 0" rpy="-${pi/2} 0 0"/>
+        <origin xyz="-0.08 0.1145 0" rpy="-${pi/2} 0 0"/>
         <axis xyz="0 0 1"/>
     </joint>
@@ -130,7 +130,7 @@
             <mass value="0.17"/>
             <inertia
-                ixx="${(1/12) * 0.17 * (3*0.06*0.06 + 0.06*0.06)}" ixy="0.0" ixz="0.0"
-                iyy="${(1/12) * 0.17 * (3*0.06*0.06 + 0.06*0.06)}" iyz="0.0"
-                izz="${(1/12) * 0.17 * (0.06*0.06)}"
+                ixx="${0.17*(3*0.06*0.06+0.06*0.06)/12}" ixy="0.0" ixz="0.0"
+                iyy="${0.17*(3*0.06*0.06+0.06*0.06)/12}" iyz="0.0"
+                izz="${0.17*(0.06*0.06)/2}"
             />
         </inertial>
@@ -142,5 +142,5 @@
         <parent link="chassis"/>
         <child link="back_right_wheel"/>
-        <origin xyz="0.08 -0.1145 0" rpy="${pi/2} 0 0"/>
+        <origin xyz="-0.08 -0.1145 0" rpy="${pi/2} 0 0"/>
         <axis xyz="0 0 -1"/>
     </joint>
@@ -162,7 +162,7 @@
             <mass value="0.17"/>
             <inertia
-                ixx="${(1/12) * 0.17 * (3*0.06*0.06 + 0.06*0.06)}" ixy="0.0" ixz="0.0"
-                iyy="${(1/12) * 0.17 * (3*0.06*0.06 + 0.06*0.06)}" iyz="0.0"
-                izz="${(1/12) * 0.17 * (0.06*0.06)}"
+                ixx="${0.17*(3*0.06*0.06+0.06*0.06)/12}" ixy="0.0" ixz="0.0"
+                iyy="${0.17*(3*0.06*0.06+0.06*0.06)/12}" iyz="0.0"
+                izz="${0.17*(0.06*0.06)/2}"
             />
         </inertial>

File: src/description/ros2_control.xacro (robot description, xacro)
@@ -37,5 +37,5 @@
 			<state_interface name="position"></state_interface>
 		</joint>
-	</ros2_control>
+		</ros2_control>
 	<gazebo>
 		<plugin name="gazebo_ros2_control" filename="libgazebo_ros2_control.so">
